File: SharpBreakout.kicad_sch (KiCad schematic)
At the start: 14 parts, among them J1 Conn_01x21_MountingPin, J2 Conn_01x02_Pin, J3 Conn_02x10_Odd_Even, J4 Conn_02x02_Odd_Even, J5 Conn_02x10_Odd_Even, J6 Conn_01x02_Pin, U1 SiP32431DR3, U2 SiP32431DR3

Commit message: Added README and pinout
Parts:
- J1: value Conn_01x21_MountingPin -> Molex 503566-2102
Other:
- company: (none) -> Helmut Lord :D
- title: (none) -> Sharp Memory-in-Pixel RGB Breakout
- moved on the sheet: C1, C2, C3, C4, C5, C6, J1, J3, J4, J5, U1, U2

Commit message: Updated pinout for better performance, all colors on one GPIO periphral, all horizontal controls on same GPIO peripheral, all vertical controls on same GPIO peripheral
Parts:
- U1, U2: value SiP32431DR3 -> SiP32432DR3; symbol Power_Management:SiP32431DR3 -> Power_Management:SiP32432DR3
Connections:
- net B0: now also J5.10 (Pin_10); no longer J5.18 (Pin_18)
- net B1: now also J5.11 (Pin_11); no longer J3.6 (Pin_6)
- net BCK: now also J3.4 (Pin_4); no longer J3.3 (Pin_3)
- net BSP: now also J3.5 (Pin_5); no longer J5.13 (Pin_13)
- net G0: now also J5.7 (Pin_7); no longer J5.15 (Pin_15)
- net G1: now also J5.12 (Pin_12); no longer J3.5 (Pin_5)
- net GCK: now also J5.13 (Pin_13); no longer J5.10 (Pin_10)
- net GEN: now also J5.15 (Pin_15); no longer J5.14 (Pin_14)
- net GSP: now also J5.14 (Pin_14); no longer J5.11 (Pin_11)
- net INTB: now also J5.16 (Pin_16); no longer J5.9 (Pin_9)
- net R0: now also J5.8 (Pin_8); no longer J5.16 (Pin_16)
- net R1: now also J5.9 (Pin_9); no longer J3.4 (Pin_4)
- net VA: now also J3.3 (Pin_3); no longer J5.12 (Pin_12)
- net VB: now also J3.6 (Pin_6); no longer J3.8 (Pin_8)
- net VBUS_EN: now also J5.18 (Pin_18); no longer J5.8 (Pin_8)
- net VDDIO_EN: now also J3.8 (Pin_8); no longer J5.7 (Pin_7)
